Commit message: without upper plate

File: turtlebot_ds/urdf/stacks/circles.urdf.xacro (robot description, xacro)
@@ -232,36 +232,4 @@
       </collision>
     </link>
-    <turtlebot_standoff_kinect parent="plate_2_link" number="0" x_loc="-0.1024382" y_loc="0.098" z_loc="0.0032004"/>
-    <turtlebot_standoff_kinect parent="plate_2_link" number="1" x_loc="-0.1024382" y_loc="-0.098" z_loc="0.0032004"/>
-    <turtlebot_standoff_8in parent="standoff_2in_4_link" number="0" x_loc="0" y_loc="0" z_loc="0.05715"/>
-    <turtlebot_standoff_8in parent="standoff_2in_5_link" number="1" x_loc="0" y_loc="0" z_loc="0.05715"/>
-    <turtlebot_standoff_8in parent="standoff_2in_6_link" number="2" x_loc="0" y_loc="0" z_loc="0.05715"/>
-    <turtlebot_standoff_8in parent="standoff_2in_7_link" number="3" x_loc="0" y_loc="0" z_loc="0.05715"/>
-    <joint name="plate_3_joint" type="fixed">
-      <origin xyz="-0.01316 0 0.2063496" rpy="0 0 0" />
-      <parent link="plate_2_link"/>
-      <child link="plate_3_link" />
-    </joint>
-    <link name="plate_3_link">
-      <inertial>
-        <mass value="0.01" />
-        <origin xyz="0 0 0" />
-        <inertia ixx="0.0001" ixy="0.0" ixz="0.0"
-          iyy="0.0001" iyz="0.0"
-          izz="0.0001" />
-      </inertial>
-      <visual>
-        <origin xyz=" 0 0 0 " rpy="0 0 0" />
-        <geometry>
-          <mesh filename="package://turtlebot_description/meshes/stacks/circles/plate_2_logo.dae"/>
-        </geometry>
-      </visual>
-      <collision>
-        <origin xyz="0.0 0.0 0.0" rpy="0 0 0" />
-        <geometry>
-          <box size="0.288 0.315 0.006401"/>
-        </geometry>
-      </collision>
-    </link>
   </xacro:macro>
 </robot>

Commit message: just the first plate and a pin for the camera

File: turtlebot_ds/urdf/stacks/circles.urdf.xacro (robot description, xacro)
@@ -202,34 +202,5 @@
       </collision>
     </link>
-    <turtlebot_standoff_2in parent="standoff_2in_0_link" number="4" x_loc="0" y_loc="0" z_loc="0.05715"/>
-    <turtlebot_standoff_2in parent="standoff_2in_1_link" number="5" x_loc="0" y_loc="0" z_loc="0.05715"/>
-    <turtlebot_standoff_2in parent="standoff_2in_2_link" number="6" x_loc="0" y_loc="0" z_loc="0.05715"/>
-    <turtlebot_standoff_2in parent="standoff_2in_3_link" number="7" x_loc="0" y_loc="0" z_loc="0.05715"/>
-    <joint name="plate_2_joint" type="fixed">
-      <origin xyz="0 0 0.0572008" rpy="0 0 0" />
-      <parent link="plate_1_link"/>
-      <child link="plate_2_link" />
-    </joint>
-    <link name="plate_2_link">
-      <inertial>
-        <mass value="0.01" />
-        <origin xyz="0 0 0" />
-        <inertia ixx="0.001" ixy="0.0" ixz="0.0"
-          iyy="0.001" iyz="0.0"
-          izz="0.001" />
-      </inertial>
-      <visual>
-        <origin xyz=" 0 0 0 " rpy="0 0 0" />
-        <geometry>
-          <mesh filename="package://turtlebot_description/meshes/stacks/circles/plate_1_logo.dae"/>
-        </geometry>
-      </visual>
-      <collision>
-        <origin xyz="0.0 0.0 0.0" rpy="0 0 0" />
-        <geometry>
-          <box size="0.314856 0.314856 0.006401"/>
-        </geometry>
-      </collision>
-    </link>
+    <turtlebot_standoff_2in parent="standoff_2in_0_link" number="4" x_loc="0.0815" y_loc="-0.132" z_loc="0.05715"/>
   </xacro:macro>
 </robot>
