Commit message: Camera has been rotated to see the flor

File: turtlebot_ds/robots/kobukids.urdf.xacro (robot description, xacro)
@@ -19,5 +19,5 @@
     <xacro:include filename="$(find hector_sensors_description)/urdf/generic_camera.urdf.xacro" />
     <xacro:generic_camera name="front_cam" parent="base_link" ros_topic="camera/image" cam_info_topic="camera/camera_info" update_rate="10" res_x="320" res_y="240" image_format="R8G8B8" hfov="90">
-      <origin xyz="0.2 0.0 0.1" rpy="0 0 0"/>
+      <origin xyz="0.18 0.0 0.1" rpy="0 0.7854 0"/>
     </xacro:generic_camera>
 </robot>

Commit message: hexagon is added to put the laser and the camera.

File: turtlebot_ds/robots/kobukids.urdf.xacro (robot description, xacro)
@@ -6,18 +6,17 @@
 -->
 <robot name="turtlebot" xmlns:xacro="http://ros.org/wiki/xacro">
-  <xacro:include filename="$(find turtlebot_description)/urdf/turtlebot_library.urdf.xacro" />
-  <kobuki/>
-<!--
-  stack_hexagons parent="base_link"
--->
- <!-- Hokuyo UTM-30LX mounted upside down below the quadrotor body -->
+	<xacro:include filename="$(find turtlebot_description)/urdf/turtlebot_library.urdf.xacro" />
+	<xacro:include filename="$(find turtlebot_ds)/urdf/stacks/hexagon.urdf.xacro" />
+	<kobuki/>
+	<stack_hexagon parent="base_link"/>
+	<!-- Hokuyo UTM-30LX mounted upside down below the quadrotor body -->
     <xacro:include filename="$(find hector_sensors_description)/urdf/hokuyo_utm30lx.urdf.xacro" />
     <xacro:hokuyo_utm30lx name="laser0" parent="base_link" ros_topic="scan" update_rate="40" ray_count="1081" min_angle="-135" max_angle="135">
-      <origin xyz="0.0 0.0 0.15" rpy="0 0 0"/>
+      <origin xyz="0.0 0.0 0.18" rpy="0 0 0"/>
     </xacro:hokuyo_utm30lx>
     <!-- Forward facing camera -->
     <xacro:include filename="$(find hector_sensors_description)/urdf/generic_camera.urdf.xacro" />
     <xacro:generic_camera name="front_cam" parent="base_link" ros_topic="camera/image" cam_info_topic="camera/camera_info" update_rate="10" res_x="320" res_y="240" image_format="R8G8B8" hfov="90">
-      <origin xyz="0.18 0.0 0.1" rpy="0 0.7854 0"/>
+      <origin xyz="0.165 0.0 0.134" rpy="0 0.7854 0"/>
     </xacro:generic_camera>
 </robot>

Commit message: moving up the camera

File: turtlebot_ds/robots/kobukids.urdf.xacro (robot description, xacro)
@@ -18,5 +18,5 @@
     <xacro:include filename="$(find hector_sensors_description)/urdf/generic_camera.urdf.xacro" />
     <xacro:generic_camera name="front_cam" parent="base_link" ros_topic="camera/image" cam_info_topic="camera/camera_info" update_rate="10" res_x="320" res_y="240" image_format="R8G8B8" hfov="90">
-      <origin xyz="0.165 0.0 0.134" rpy="0 0.7854 0"/>
+      <origin xyz="0.16 0.0 0.17" rpy="0 0.7854 0"/>
     </xacro:generic_camera>
 </robot>

Commit message: comments and tabulations

File: turtlebot_ds/robots/kobukids.urdf.xacro (robot description, xacro)
@@ -8,15 +8,21 @@
 	<xacro:include filename="$(find turtlebot_description)/urdf/turtlebot_library.urdf.xacro" />
 	<xacro:include filename="$(find turtlebot_ds)/urdf/stacks/hexagon.urdf.xacro" />
+	<!-- Robot base -->
 	<kobuki/>
+	<!-- Hexagon base -->
 	<stack_hexagon parent="base_link"/>
-	<!-- Hokuyo UTM-30LX mounted upside down below the quadrotor body -->
+	<!-- Hokuyo UTM-30LX -->
     <xacro:include filename="$(find hector_sensors_description)/urdf/hokuyo_utm30lx.urdf.xacro" />
-    <xacro:hokuyo_utm30lx name="laser0" parent="base_link" ros_topic="scan" update_rate="40" ray_count="1081" min_angle="-135" max_angle="135">
-      <origin xyz="0.0 0.0 0.18" rpy="0 0 0"/>
+    <xacro:hokuyo_utm30lx name="laser0" parent="base_link" ros_topic="scan"
+			update_rate="40" ray_count="1081" min_angle="-135" max_angle="135">
+    		<origin xyz="0.0 0.0 0.18" rpy="0 0 0"/>
     </xacro:hokuyo_utm30lx>
     <!-- Forward facing camera -->
     <xacro:include filename="$(find hector_sensors_description)/urdf/generic_camera.urdf.xacro" />
-    <xacro:generic_camera name="front_cam" parent="base_link" ros_topic="camera/image" cam_info_topic="camera/camera_info" update_rate="10" res_x="320" res_y="240" image_format="R8G8B8" hfov="90">
-      <origin xyz="0.16 0.0 0.17" rpy="0 0.7854 0"/>
+    <xacro:generic_camera name="front_cam" parent="base_link" ros_topic="camera/image"
+			cam_info_topic="camera/camera_info" update_rate="10" res_x="320" res_y="240"
+			image_format="R8G8B8" hfov="90">
+		<!-- Rotated 45 degress pointing to the floor -->
+	    <origin xyz="0.16 0.0 0.17" rpy="0 0.7854 0"/>
     </xacro:generic_camera>
 </robot>

Commit message: camera mounted on a bar

File: turtlebot_ds/robots/kobukids.urdf.xacro (robot description, xacro)
@@ -24,5 +24,5 @@
 			image_format="R8G8B8" hfov="90">
 		<!-- Rotated 45 degress pointing to the floor -->
-	    <origin xyz="0.16 0.0 0.17" rpy="0 0.7854 0"/>
+	    <origin xyz="0.155 0.0 0.185" rpy="0 0.7854 0"/>
     </xacro:generic_camera>
 </robot>

File: turtlebot_ds/urdf/stacks/hexagon.urdf.xacro (robot description, xacro)
@@ -31,4 +31,32 @@
         <mass value="0.001"/>
         <origin xyz="0 0 0" rpy="0 0 0"/>
+        <inertia ixx="0.0001" ixy="0.0" ixz="0.0"
+                 iyy="0.0001" iyz="0.0"
+                 izz="0.0001"/>
+      </inertial>
+    </link>
+  </xacro:macro>
+  <xacro:macro name="stack_middle_pole" params="parent number x_loc y_loc z_loc">
+    <joint name="pole_middle_${number}_joint" type="fixed">
+      <origin xyz="${x_loc} ${y_loc} ${z_loc}" rpy="0 0 0" />
+      <parent link="${parent}"/>
+      <child link="pole_middle_${number}_link"/>
+    </joint>
+    <link name="pole_middle_${number}_link">
+      <visual>
+        <origin xyz="0 0 0" rpy="0 ${M_PI} 0"/>
+        <geometry>
+          <mesh filename="package://turtlebot_description/meshes/stacks/hexagons/pole_middle.dae"/>
+        </geometry>
+      </visual>
+      <collision>
+        <origin xyz="0 0 0" rpy="0 0 0"/>
+        <geometry>
+          <cylinder length="0.0608" radius=".006"/>
+        </geometry>
+      </collision>
+      <inertial>
+        <mass value="0.001"/>
+        <origin xyz="0 0 0"/>
         <inertia ixx="0.0001" ixy="0.0" ixz="0.0"
                  iyy="0.0001" iyz="0.0"
@@ -75,4 +103,5 @@
       </inertial>
     </link>
+    <stack_middle_pole parent="${parent}" number="0" x_loc= "0.145" y_loc= "0.0" z_loc="0.1650"/>
   </xacro:macro>
 </robot>

Commit message: - new robot drawer - migrating to indigo

File: turtlebot_ds/robots/kobukids.urdf.xacro (robot description, xacro)
@@ -19,9 +19,9 @@
  	 <stack_circles parent="base_link"/>
 	<!-- Hokuyo UTM-30LX -->
-    <xacro:include filename="$(find hector_sensors_description)/urdf/hokuyo_utm30lx.urdf.xacro" />
-    <xacro:hokuyo_utm30lx name="laser0" parent="base_link" ros_topic="scan"
-			update_rate="40" ray_count="1081" min_angle="-135" max_angle="135">
-    		<origin xyz="0.0 0.0 0.18" rpy="0 0 0"/>
-    </xacro:hokuyo_utm30lx>
+    <!--<xacro:include filename="$(find hector_sensors_description)/urdf/hokuyo_utm30lx.urdf.xacro" />-->
+    <!--<xacro:hokuyo_utm30lx name="laser0" parent="base_link" ros_topic="scan"-->
+			<!--update_rate="40" ray_count="1081" min_angle="-135" max_angle="135">-->
+    		<!--<origin xyz="0.0 0.0 0.18" rpy="0 0 0"/>-->
+    <!--</xacro:hokuyo_utm30lx>-->
     <!-- Forward facing camera -->
     <xacro:include filename="$(find hector_sensors_description)/urdf/generic_camera.urdf.xacro" />
